File: wemos-mains-dev.kicad_pcb (KiCad board)
At the start: 2 copper layers, 74.2 x 46.5 mm, 16 parts, among them J1 Screw_Terminal_01x02, J2 Conn_01x08, J3 Conn_01x08, J8 SDA, J9 SDA, U1 AC-05-3, U2 WeMos_D1_mini

Commit message: Changed pinheader for breakout to 02x12
Parts:
- removed J3: Conn_01x08, Connector_PinHeader_2.54mm:PinHeader_1x12_P2.54mm_Vertical
- J2: value Conn_01x08 -> Conn_02x12_Odd_Even; footprint Connector_PinHeader_2.54mm:PinHeader_1x12_P2.54mm_Vertical -> Connector_PinHeader_2.54mm:PinHeader_2x12_P2.54mm_Vertical
- J8, J9: value SDA -> SDA PU
- moved J2 27.8 mm to (134.6, 87.1), turned to 0 degrees
- moved C2 7.62 mm to (139.7, 104.1)
Connections:
- J2 pad 1: +5V -> D0_GPIO
- J2 pad 10: TX -> D7_MOSI
- J2 pad 11: RX -> D5_SCK
- J2 pad 12: D0_GPIO -> D8_CS
- J2 pad 3: D3_ONE -> RX
- J2 pad 4: GND -> D1_SCL
- J2 pad 5: A0_ANL -> TX
- J2 pad 6: +3V3 -> D2_SDA
- J2 pad 7: D5_SCK -> GND
- J2 pad 8: D6_MISO -> GND
- J2 pad 9: GND -> D6_MISO
Routing:
- net GND: track 5.90 -> 0.00 mm
- net D8_CS: track 14.1 -> 19.2 mm
- net D7_MOSI: track 14.5 -> 11.5 mm
- net D2_SDA: track 71.6 -> 72.9 mm
- net D1_SCL: track 62.2 -> 63.5 mm
- net RST: track 13.6 -> 12.3 mm
- net +5V: track 76.5 -> 75.3 mm
- net D4_LED: track 42.5 -> 41.3 mm
- net RX: track 53.9 -> 55.0 mm
Other:
- board text added: "SCL"
- board text added: "SDA"
